File: BatteryBoardV1/BatteryCharger.sch (KiCad schematic (older format))
At the start: 10 parts, among them U1 MCP73213

Commit message: Add files via upload
Parts:
- JIn1: footprint BJCs:DC_2.1mm_CUI-PJ-202A -> Connectors:Barrel_Jack_CUI_PJ-102AH
- Q1: renamed from Q?; footprint (none) -> TO_SOT_Packages_SMD:SOT-23
Connections:
- net GND: now also Q1.2 (S), Q1.3 (D)
- net at C1.1, JOut1.1 (Pin_1), U1.3 (VBAT)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: now also Q1.1 (G)
Other:
- moved on the sheet: Q1
Changed lines of the file:
@@
 LIBS:BatCharge
 LIBS:Connectors
+LIBS:dk_Addressable-Specialty
+LIBS:dk_Alarms-Buzzers-and-Sirens
+LIBS:dk_Automotive-Relays
+LIBS:dk_Balun
+LIBS:dk_Barrel-Audio-Connectors
+LIBS:dk_Battery-Holders-Clips-Contacts
+LIBS:dk_Clock-Timing-Clock-Generators-PLLs-Frequency-Synthesizers
+LIBS:dk_Clock-Timing-Programmable-Timers-and-Oscillators
+LIBS:dk_Clock-Timing-Real-Time-Clocks
+LIBS:dk_Coaxial-Connectors-RF
+LIBS:dk_Current-Transducers
+LIBS:dk_Data-Acquisition-ADCs-DACs-Special-Purpose
+LIBS:dk_Data-Acquisition-Analog-to-Digital-Converters-ADC
+LIBS:dk_Data-Acquisition-Digital-Potentiometers
+LIBS:dk_Data-Acquisition-Digital-to-Analog-Converters-DAC
+LIBS:dk_Data-Acquisition-Touch-Screen-Controllers
+LIBS:dk_DC-DC-Converters
+LIBS:dk_Digital-Isolators
+LIBS:dk_Diodes-Bridge-Rectifiers
+LIBS:dk_Diodes-Rectifiers-Arrays
+LIBS:dk_Diodes-Rectifiers-Single
+LIBS:dk_Diodes-Zener-Single
+LIBS:dk_Display-Modules-LED-Character-and-Numeric
+LIBS:dk_D-Sub-Connectors
+LIBS:dk_Embedded-Microcontrollers
+LIBS:dk_Encoders
+LIBS:dk_Evaluation-Boards-Sensors
+LIBS:dk_Ferrite-Beads-and-Chips
+LIBS:dk_Fixed-Inductors
+LIBS:dk_Fuses
+LIBS:dk_Gas-Sensors
+LIBS:dk_Humidity-Moisture-Sensors
+LIBS:dk_Image-Sensors-Camera
+LIBS:dk_Infrared-UV-Visible-Emitters
+LIBS:dk_Inrush-Current-Limiters-ICL
+LIBS:dk_Interface-Analog-Switches-Multiplexers-Demultiplexers
+LIBS:dk_Interface-Analog-Switches-Special-Purpose
+LIBS:dk_Interface-Controllers
+LIBS:dk_Interface-Drivers-Receivers-Transceivers
+LIBS:dk_Interface-I-O-Expanders
+LIBS:dk_Interface-Modules
+LIBS:dk_Interface-Sensor-and-Detector-Interfaces
+LIBS:dk_Interface-Sensor-Capacitive-Touch
+LIBS:dk_Interface-Specialized
+LIBS:dk_LED-Indication-Discrete
+LIBS:dk_LEDs-Circuit-Board-Indicators-Arrays-Light-Bars-Bar-Graphs
+LIBS:dk_Linear-Amplifiers-Audio
+LIBS:dk_Linear-Amplifiers-Instrumentation-OP-Amps-Buffer-Amps
+LIBS:dk_Linear-Comparators
+LIBS:dk_Logic-Buffers-Drivers-Receivers-Transceivers
+LIBS:dk_Logic-Flip-Flops
+LIBS:dk_Logic-Gates-and-Inverters
+LIBS:dk_Logic-Multivibrators
+LIBS:dk_Logic-Shift-Registers
+LIBS:dk_Logic-Signal-Switches-Multiplexers-Decoders
+LIBS:dk_Logic-Translators-Level-Shifters
+LIBS:dk_Magnetic-Sensors-Compass-Magnetic-Field-Modules
+LIBS:dk_Magnetic-Sensors-Linear-Compass-ICs
+LIBS:dk_Magnetic-Sensors-Switches-Solid-State
+LIBS:dk_Memory
+LIBS:dk_Memory-Connectors-PC-Card-Sockets
+LIBS:dk_Microphones
+LIBS:dk_Modular-Connectors-Jacks
+LIBS:dk_Modular-Connectors-Jacks-With-Magnetics
+LIBS:dk_Motion-Sensors-Accelerometers
+LIBS:dk_Motion-Sensors-IMUs-Inertial-Measurement-Units
+LIBS:dk_Motion-Sensors-Tilt-Switches
+LIBS:dk_Navigation-Switches-Joystick
+LIBS:dk_Optical-Sensors-Ambient-Light-IR-UV-Sensors
+LIBS:dk_Optical-Sensors-Photo-Detectors-Remote-Receiver
+LIBS:dk_Optical-Sensors-Photodiodes
+LIBS:dk_Optical-Sensors-Phototransistors
+LIBS:dk_Optical-Sensors-Reflective-Analog-Output
+LIBS:dk_Optoisolators-Logic-Output
+LIBS:dk_Optoisolators-Transistor-Photovoltaic-Output
+LIBS:dk_Optoisolators-Triac-SCR-Output
+LIBS:dk_Oscillators
+LIBS:dk_PMIC-AC-DC-Converters-Offline-Switchers
+LIBS:dk_PMIC-Battery-Chargers
+LIBS:dk_PMIC-Battery-Management
+LIBS:dk_PMIC-Current-Regulation-Management
+LIBS:dk_PMIC-Full-Half-Bridge-Drivers
+LIBS:dk_PMIC-Gate-Drivers
+LIBS:dk_PMIC-LED-Drivers
+LIBS:dk_PMIC-Motor-Drivers-Controllers
+LIBS:dk_PMIC-OR-Controllers-Ideal-Diodes
+LIBS:dk_PMIC-Power-Distribution-Switches-Load-Drivers
+LIBS:dk_PMIC-Power-Management-Specialized
+LIBS:dk_PMIC-RMS-to-DC-Converters
+LIBS:dk_PMIC-Supervisors
+LIBS:dk_PMIC-Thermal-Management
+LIBS:dk_PMIC-V-F-and-F-V-Converters
+LIBS:dk_PMIC-Voltage-Reference
+LIBS:dk_PMIC-Voltage-Regulators-DC-DC-Switching-Controllers
+LIBS:dk_PMIC-Voltage-Regulators-DC-DC-Switching-Regulators
+LIBS:dk_PMIC-Voltage-Regulators-Linear
+LIBS:dk_PMIC-Voltage-Regulators-Special-Purpose
+LIBS:dk_Power-Relays-Over-2-Amps
+LIBS:dk_Pressure-Sensors-Transducers
+LIBS:dk_Programmable-Oscillators
+LIBS:dk_Pushbutton-Switches
+LIBS:dk_Rectangular-Connectors-Headers-Male-Pins
+LIBS:dk_Reed-Relays
+LIBS:dk_Resistor-Networks-Arrays
+LIBS:dk_RF-Amplifiers
+LIBS:dk_RF-Antennas
+LIBS:dk_RF-Demodulators
+LIBS:dk_RF-Detectors
+LIBS:dk_RF-Evaluation-and-Development-Kits-Boards
+LIBS:dk_RFID-RF-Access-Monitoring-ICs
+LIBS:dk_RF-Receivers
+LIBS:dk_RF-Switches
+LIBS:dk_RF-Transceiver-ICs
+LIBS:dk_RF-Transceiver-Modules
+LIBS:dk_RF-Transmitters
+LIBS:dk_Rotary-Potentiometers-Rheostats
+LIBS:dk_Sensors-Transducers_Accessories
+LIBS:dk_Signal-Relays-Up-to-2-Amps
+LIBS:dk_Slide-Switches
+LIBS:dk_Solid-State-Relays
+LIBS:dk_Specialized-ICs
+LIBS:dk_Specialized-Sensors
+LIBS:dk_Surge-Suppression-ICs
+LIBS:dk_Tactile-Switches
+LIBS:dk_Temperature-Sensors-Analog-and-Digital-Output
+LIBS:dk_Thermal-Cutoffs-Thermal-Fuses
+LIBS:dk_Thyristors-DIACs-SIDACs
+LIBS:dk_Thyristors-SCRs
+LIBS:dk_Thyristors-TRIACs
+LIBS:dk_Toggle-Switches
+LIBS:dk_Transistors-Bipolar-BJT-Arrays
+LIBS:dk_Transistors-Bipolar-BJT-RF
+LIBS:dk_Transistors-Bipolar-BJT-Single
+LIBS:dk_Transistors-Bipolar-BJT-Single-Pre-Biased
+LIBS:dk_Transistors-FETs-MOSFETs-Arrays
+LIBS:dk_Transistors-FETs-MOSFETs-RF
+LIBS:dk_Transistors-FETs-MOSFETs-Single
+LIBS:dk_Transistors-JFETs
+LIBS:dk_Trimmer-Potentiometers
+LIBS:dk_TVS-Diodes
+LIBS:dk_TVS-Mixed-Technology
+LIBS:dk_USB-DVI-HDMI-Connectors
 LIBS:BatteryCharger-cache
 EELAYER 25 0
@@
 VBAT-
 $Comp
-L VDD #PWR07
+L VDD #PWR06
 U 1 1 5A8B7E71
 P 2400 3750
-F 0 "#PWR07" H 2400 3600 50  0001 C CNN
+F 0 "#PWR06" H 2400 3600 50  0001 C CNN
 F 1 "VDD" H 2400 3900 50  0000 C CNN
 F 2 "" H 2400 3750 50  0001 C CNN
@@
 F 0 "JIn1" H 1600 4060 50  0000 C CNN
 F 1 "Barrel_Jack" H 1600 3675 50  0000 C CNN
-F 2 "BJCs:DC_2.1mm_CUI-PJ-202A" H 1650 3810 50  0001 C CNN
+F 2 "Connectors:Barrel_Jack_CUI_PJ-102AH" H 1650 3810 50  0001 C CNN
 F 3 "" H 1650 3810 50  0001 C CNN
 	1    1600 3850
@@
 $EndComp
 $Comp
-L GND #PWR09
+L GND #PWR07
 U 1 1 5A8B89FB
 P 2200 4050
-F 0 "#PWR09" H 2200 3800 50  0001 C CNN
+F 0 "#PWR07" H 2200 3800 50  0001 C CNN
 F 1 "GND" H 2200 3900 50  0000 C CNN
 F 2 "" H 2200 4050 50  0001 C CNN
@@
 	0    1    1    0
 $EndComp
+$Comp
+L Q_NMOS_GSD Q1
+U 1 1 5A9AF155
+P 5925 6150
+F 0 "Q1" H 6125 6200 50  0000 L CNN
+F 1 "Q_NMOS_GSD" H 6125 6100 50  0000 L CNN
+F 2 "TO_SOT_Packages_SMD:SOT-23" H 6125 6250 50  0001 C CNN
+F 3 "" H 5925 6150 50  0001 C CNN
+	1    5925 6150
+	0    1    1    0
+$EndComp
 Wire Wire Line
 	5950 4550 5950 4875
@@
 Wire Wire Line
 	2325 4775 2150 4775
-$Comp
-L Q_NMOS_GSD Q?
-U 1 1 5A9AF155
-P 2775 4075
-F 0 "Q?" H 2975 4125 50  0000 L CNN
-F 1 "Q_NMOS_GSD" H 2975 4025 50  0000 L CNN
-F 2 "" H 2975 4175 50  0001 C CNN
-F 3 "" H 2775 4075 50  0001 C CNN
-	1    2775 4075
-	0    -1   -1   0
+Wire Wire Line
+	5925 5950 5925 5800
+Wire Wire Line
+	5925 5800 5750 5800
+Wire Wire Line
+	5750 5800 5750 5600
+Connection ~ 5750 5600
+Wire Wire Line
+	6125 6250 6125 5600
+Connection ~ 6125 5600
+$Comp
+L GND #PWR08
+U 1 1 5AA857E4
+P 5725 6250
+F 0 "#PWR08" H 5725 6000 50  0001 C CNN
+F 1 "GND" H 5725 6100 50  0000 C CNN
+F 2 "" H 5725 6250 50  0001 C CNN
+F 3 "" H 5725 6250 50  0001 C CNN
+	1    5725 6250
+	0    1    1    0
 $EndComp
 $EndSCHEMATC

Commit message: Add files via upload
Parts:
- R1: value 1.185K -> 3K
Connections:
- net GND: no longer JOut1.2 (Pin_2), Q1.3 (D)
- net VBAT+: now also C1.1, JOut1.1 (Pin_1), Q1.1 (G), U1.3 (VBAT), U1.4 (VBAT)
- new net VBAT-: JOut1.2 (Pin_2), Q1.3 (D)
Other:
- moved on the sheet: Q1
Changed lines of the file:
@@
 encoding utf-8
 Sheet 1 1
-Title ""
+Title "Battery Charger Circuit"
 Date ""
 Rev ""
-Comp ""
-Comment1 ""
+Comp "Student Organization for Aerospace Research"
+Comment1 "By: Prithvi Shankara and Evan Wilkinson"
 Comment2 ""
 Comment3 ""
@@
 P 7000 3750
 F 0 "R1" V 7080 3750 50  0000 C CNN
-F 1 "1.185K" V 7000 3750 50  0000 C CNN
+F 1 "3K" V 7000 3750 50  0000 C CNN
 F 2 "Resistors_SMD:R_0603_HandSoldering" V 6930 3750 50  0001 C CNN
 F 3 "" H 7000 3750 50  0001 C CNN
@@
 U 1 1 5A8B62D4
 P 5875 5400
-F 0 "JOut1" H 5875 5500 50  0000 C CNN
+F 0 "JOut1" V 5875 5575 50  0000 C CNN
 F 1 "Bat.Terms." V 5975 5350 50  0000 C CNN
 F 2 "Connectors_Terminal_Blocks:TerminalBlock_Altech_AK300-2_P5.00mm" H 5875 5400 50  0001 C CNN
@@
 	0    -1   -1   0
 $EndComp
-Text Label 5725 5575 2    60   ~ 0
+Text Label 5800 5600 2    60   ~ 0
 VBAT+
-Text Label 6325 5500 1    60   ~ 0
+Text Label 6275 5600 2    60   ~ 0
 VBAT-
 $Comp
@@
 L Q_NMOS_GSD Q1
 U 1 1 5A9AF155
-P 5925 6150
-F 0 "Q1" H 6125 6200 50  0000 L CNN
-F 1 "Q_NMOS_GSD" H 6125 6100 50  0000 L CNN
-F 2 "TO_SOT_Packages_SMD:SOT-23" H 6125 6250 50  0001 C CNN
-F 3 "" H 5925 6150 50  0001 C CNN
-	1    5925 6150
-	0    1    1    0
+P 6500 5700
+F 0 "Q1" V 6800 5650 50  0000 L CNN
+F 1 "Q_NMOS_GSD" V 6725 5450 50  0000 L CNN
+F 2 "TO_SOT_Packages_SMD:SOT-23" H 6700 5800 50  0001 C CNN
+F 3 "" H 6500 5700 50  0001 C CNN
+	1    6500 5700
+	0    -1   -1   0
 $EndComp
 Wire Wire Line
 	5950 4550 5950 4875
 Wire Wire Line
-	5950 4750 6325 4750
+	5950 4750 7025 4750
 Connection ~ 5950 4750
 Wire Wire Line
@@
 	4800 3075 4800 3750
 Connection ~ 4800 3750
-Connection ~ 6775 4125
-Wire Wire Line
-	6325 4750 6325 5600
-Wire Wire Line
-	6325 5600 5975 5600
 Wire Wire Line
 	4800 4125 4800 5600
@@
 	2325 4775 2150 4775
 Wire Wire Line
-	5925 5950 5925 5800
-Wire Wire Line
-	5925 5800 5750 5800
-Wire Wire Line
-	5750 5800 5750 5600
-Connection ~ 5750 5600
-Wire Wire Line
-	6125 6250 6125 5600
-Connection ~ 6125 5600
-$Comp
-L GND #PWR08
-U 1 1 5AA857E4
-P 5725 6250
-F 0 "#PWR08" H 5725 6000 50  0001 C CNN
-F 1 "GND" H 5725 6100 50  0000 C CNN
-F 2 "" H 5725 6250 50  0001 C CNN
-F 3 "" H 5725 6250 50  0001 C CNN
-	1    5725 6250
-	0    1    1    0
-$EndComp
+	5975 5600 6300 5600
+Wire Wire Line
+	7025 4750 7025 5600
+Wire Wire Line
+	7025 5600 6700 5600
+Wire Wire Line
+	6500 5900 5450 5900
+Wire Wire Line
+	5450 5900 5450 5600
+Connection ~ 5450 5600
 $EndSCHEMATC

Commit message: Add files via upload
Parts:
- added J1: Conn_01x04_Male, Connector_Molex:Molex_Micro-Fit_3.0_43045-0412_2x02_P3.00mm_Vertical, symbol Conn_01x04_Male
- D1: footprint LEDs:LED_0603_HandSoldering -> LEDs:LED_0805_HandSoldering
- JIn2, JOut1: footprint Connectors_Terminal_Blocks:TerminalBlock_Altech_AK300-2_P5.00mm -> TerminalBlock_Phoenix:TerminalBlock_Phoenix_PT-1,5-2-5.0-H_1x02_P5.00mm_Horizontal
- R1, R2: footprint Resistors_SMD:R_0603_HandSoldering -> Resistors_SMD:R_0805_HandSoldering
- U1: footprint Housings_SSOP:MSOP-10-1EP_3x3mm_Pitch0.5mm -> Housings_DFN_QFN:DFN-10-1EP_3x3mm_Pitch0.5mm
Connections:
- net GND: now also J1.1 (Pin_1), J1.2 (Pin_2)
- net VBAT+: now also J1.4 (Pin_4)
- net VDD: now also J1.3 (Pin_3)
- no-connect marks 0 -> 2
Other:
- note added: "8.4V regulated voltage"
- note added: "Battery Specifications"
- note added: "Datasheet of Charging IC\n"
- note added: "Dual-cell Li-ion/Li-polymer battery"
- note added: "Maximum Input Voltage: 16V\n"
- note added: "Minimum Input Voltage: 4V"
- note added: "Not Connected"
- note added: "Regulated Current through 3K Resistor: 400mA"
- note added: "Supply Specifications"
- note added: "https://www.mouser.com/ds/2/268/22190a-13379.pdf"
- moved on the sheet: Q1
Changed lines of the file:
@@
 Date ""
 Rev ""
-Comp "Student Organization for Aerospace Research"
-Comment1 "By: Prithvi Shankara and Evan Wilkinson"
-Comment2 ""
+Comp "SOAR"
+Comment1 "Evan Wilkinson"
+Comment2 "Prithvi Shankara"
 Comment3 ""
 Comment4 ""
@@
 F 0 "U1" H 5950 4450 60  0000 C CNN
 F 1 "MCP73213" H 5950 4550 60  0000 C CNN
-F 2 "Housings_SSOP:MSOP-10-1EP_3x3mm_Pitch0.5mm" H 5900 3950 60  0001 C CNN
+F 2 "Housings_DFN_QFN:DFN-10-1EP_3x3mm_Pitch0.5mm" H 5900 3950 60  0001 C CNN
 F 3 "" H 5900 3950 60  0001 C CNN
 	1    5950 4000
@@
 F 0 "R1" V 7080 3750 50  0000 C CNN
 F 1 "3K" V 7000 3750 50  0000 C CNN
-F 2 "Resistors_SMD:R_0603_HandSoldering" V 6930 3750 50  0001 C CNN
+F 2 "Resistors_SMD:R_0805_HandSoldering" V 6930 3750 50  0001 C CNN
 F 3 "" H 7000 3750 50  0001 C CNN
 	1    7000 3750
@@
 F 0 "R2" V 7205 4125 50  0000 C CNN
 F 1 "1K" V 7125 4125 50  0000 C CNN
-F 2 "Resistors_SMD:R_0603_HandSoldering" V 7055 4125 50  0001 C CNN
+F 2 "Resistors_SMD:R_0805_HandSoldering" V 7055 4125 50  0001 C CNN
 F 3 "" H 7125 4125 50  0001 C CNN
 	1    7125 4125
@@
 F 0 "D1" H 7800 4225 50  0000 C CNN
 F 1 "LED" H 7800 4025 50  0000 C CNN
-F 2 "LEDs:LED_0603_HandSoldering" H 7800 4125 50  0001 C CNN
+F 2 "LEDs:LED_0805_HandSoldering" H 7800 4125 50  0001 C CNN
 F 3 "" H 7800 4125 50  0001 C CNN
 	1    7800 4125
@@
 P 4100 3750
 F 0 "#PWR05" H 4100 3600 50  0001 C CNN
-F 1 "VDD" H 4100 3900 50  0000 C CNN
+F 1 "VDD" V 4100 3950 50  0000 C CNN
 F 2 "" H 4100 3750 50  0001 C CNN
 F 3 "" H 4100 3750 50  0001 C CNN
@@
 F 0 "JOut1" V 5875 5575 50  0000 C CNN
 F 1 "Bat.Terms." V 5975 5350 50  0000 C CNN
-F 2 "Connectors_Terminal_Blocks:TerminalBlock_Altech_AK300-2_P5.00mm" H 5875 5400 50  0001 C CNN
+F 2 "TerminalBlock_Phoenix:TerminalBlock_Phoenix_PT-1,5-2-5.0-H_1x02_P5.00mm_Horizontal" H 5875 5400 50  0001 C CNN
 F 3 "" H 5875 5400 50  0001 C CNN
 	1    5875 5400
@@
 Text Label 5800 5600 2    60   ~ 0
 VBAT+
-Text Label 6275 5600 2    60   ~ 0
+Text Label 6300 5600 2    60   ~ 0
 VBAT-
 $Comp
@@
 P 2400 3750
 F 0 "#PWR06" H 2400 3600 50  0001 C CNN
-F 1 "VDD" H 2400 3900 50  0000 C CNN
+F 1 "VDD" V 2400 3950 50  0000 C CNN
 F 2 "" H 2400 3750 50  0001 C CNN
 F 3 "" H 2400 3750 50  0001 C CNN
@@
 F 0 "JIn2" H 2150 5075 50  0000 C CNN
 F 1 "Input Terms." V 2250 4925 50  0000 C CNN
-F 2 "Connectors_Terminal_Blocks:TerminalBlock_Altech_AK300-2_P5.00mm" H 2150 4975 50  0001 C CNN
+F 2 "TerminalBlock_Phoenix:TerminalBlock_Phoenix_PT-1,5-2-5.0-H_1x02_P5.00mm_Horizontal" H 2150 4975 50  0001 C CNN
 F 3 "" H 2150 4975 50  0001 C CNN
 	1    2150 4975
@@
 L Q_NMOS_GSD Q1
 U 1 1 5A9AF155
-P 6500 5700
-F 0 "Q1" V 6800 5650 50  0000 L CNN
-F 1 "Q_NMOS_GSD" V 6725 5450 50  0000 L CNN
-F 2 "TO_SOT_Packages_SMD:SOT-23" H 6700 5800 50  0001 C CNN
-F 3 "" H 6500 5700 50  0001 C CNN
-	1    6500 5700
-	0    -1   -1   0
-$EndComp
+P 6525 5700
+F 0 "Q1" V 6850 5650 50  0000 L CNN
+F 1 "Q_NMOS_GSD" V 6750 5475 50  0000 L CNN
+F 2 "TO_SOT_Packages_SMD:SOT-23" H 6725 5800 50  0001 C CNN
+F 3 "" H 6525 5700 50  0001 C CNN
+	1    6525 5700
+	0    -1   -1   0
+$EndComp
+NoConn ~ 6475 4250
+NoConn ~ 5400 4250
+Text Notes 6300 4325 0    39   ~ 0
+Not Connected
+Text Notes 5175 4325 0    39   ~ 0
+Not Connected
+Text Notes 1425 3000 0    60   ~ 0
+Supply Specifications
+Text Notes 1450 3125 0    39   ~ 0
+Minimum Input Voltage: 4V
+Text Notes 1450 3200 0    39   ~ 0
+Maximum Input Voltage: 16V\n
+Text Notes 3600 6100 0    59   ~ 0
+Battery Specifications
+Text Notes 3625 6225 0    39   ~ 0
+Dual-cell Li-ion/Li-polymer battery
+Text Notes 3625 6325 0    39   ~ 0
+8.4V regulated voltage
+Text Notes 6475 3575 0    39   ~ 0
+Regulated Current through 3K Resistor: 400mA
+Text Notes 4800 1975 0    60   ~ 0
+Datasheet of Charging IC\n
+Text Notes 4800 2150 0    39   ~ 0
+https://www.mouser.com/ds/2/268/22190a-13379.pdf
 Wire Wire Line
 	5950 4550 5950 4875
@@
 	4225 4375 4225 4900
 Wire Wire Line
-	6475 3750 6850 3750
-Wire Wire Line
 	7475 3875 6475 3875
 Wire Wire Line
@@
 	7475 3750 7475 3875
 Connection ~ 7475 3800
-Connection ~ 6650 3750
 Wire Wire Line
 	6475 4000 6650 4000
@@
 	4800 3075 4800 3750
 Connection ~ 4800 3750
+Connection ~ 6775 4125
+Wire Wire Line
+	6325 5600 5975 5600
 Wire Wire Line
 	4800 4125 4800 5600
@@
 	1900 3750 2400 3750
 Wire Wire Line
-	2125 3850 1900 3850
+	1900 3850 2125 3850
 Connection ~ 2325 3750
 Wire Wire Line
 	2325 3750 2325 4775
 Wire Wire Line
-	2200 4050 2200 3950
-Wire Wire Line
-	2200 3950 1900 3950
+	2200 3950 2200 4050
+Wire Wire Line
+	1900 3950 2200 3950
 Wire Wire Line
 	2050 3850 2050 4775
@@
 	2325 4775 2150 4775
 Wire Wire Line
-	5975 5600 6300 5600
-Wire Wire Line
 	7025 4750 7025 5600
 Wire Wire Line
-	7025 5600 6700 5600
-Wire Wire Line
-	6500 5900 5450 5900
-Wire Wire Line
-	5450 5900 5450 5600
-Connection ~ 5450 5600
+	7025 5600 6725 5600
+Wire Wire Line
+	6525 5900 5475 5900
+Wire Wire Line
+	5475 5900 5475 5600
+Connection ~ 5475 5600
+Wire Notes Line
+	1425 3000 2425 3000
+Wire Notes Line
+	3600 6100 4600 6100
+Wire Wire Line
+	6850 3750 6475 3750
+Wire Notes Line
+	4800 1975 5975 1975
+$Comp
+L Conn_01x04_Male J1
+U 1 1 5AC40877
+P 5225 6625
+F 0 "J1" H 5225 6825 50  0000 C CNN
+F 1 "Conn_01x04_Male" H 5225 6325 50  0000 C CNN
+F 2 "Connector_Molex:Molex_Micro-Fit_3.0_43045-0412_2x02_P3.00mm_Vertical" H 5225 6625 50  0001 C CNN
+F 3 "" H 5225 6625 50  0001 C CNN
+	1    5225 6625
+	1    0    0    -1
+$EndComp
+$Comp
+L GND #PWR08
+U 1 1 5AC409E1
+P 5425 6525
+F 0 "#PWR08" H 5425 6275 50  0001 C CNN
+F 1 "GND" V 5425 6300 50  0000 C CNN
+F 2 "" H 5425 6525 50  0001 C CNN
+F 3 "" H 5425 6525 50  0001 C CNN
+	1    5425 6525
+	0    -1   -1   0
+$EndComp
+$Comp
+L GND #PWR09
+U 1 1 5AC40A16
+P 5425 6625
+F 0 "#PWR09" H 5425 6375 50  0001 C CNN
+F 1 "GND" V 5425 6400 50  0000 C CNN
+F 2 "" H 5425 6625 50  0001 C CNN
+F 3 "" H 5425 6625 50  0001 C CNN
+	1    5425 6625
+	0    -1   -1   0
+$EndComp
+$Comp
+L VDD #PWR010
+U 1 1 5AC40AE6
+P 5425 6725
+F 0 "#PWR010" H 5425 6575 50  0001 C CNN
+F 1 "VDD" V 5425 6950 50  0000 C CNN
+F 2 "" H 5425 6725 50  0001 C CNN
+F 3 "" H 5425 6725 50  0001 C CNN
+	1    5425 6725
+	0    1    1    0
+$EndComp
+Wire Wire Line
+	5425 6825 5950 6825
+Wire Wire Line
+	5950 6825 5950 6200
+Wire Wire Line
+	5950 6200 5200 6200
+Wire Wire Line
+	5200 6200 5200 5600
+Connection ~ 5200 5600
 $EndSCHEMATC

Commit message: Add files via upload
Parts:
- J1: footprint Connector_Molex:Molex_Micro-Fit_3.0_43045-0412_2x02_P3.00mm_Vertical -> SOAR_Library:Molex_Micro-Fit_3.0_43045-0400_2x02_P3.00mm_Horizontal
Changed lines of the file:
@@
 F 0 "J1" H 5225 6825 50  0000 C CNN
 F 1 "Conn_01x04_Male" H 5225 6325 50  0000 C CNN
-F 2 "Connector_Molex:Molex_Micro-Fit_3.0_43045-0412_2x02_P3.00mm_Vertical" H 5225 6625 50  0001 C CNN
+F 2 "SOAR_Library:Molex_Micro-Fit_3.0_43045-0400_2x02_P3.00mm_Horizontal" H 5225 6625 50  0001 C CNN
 F 3 "" H 5225 6625 50  0001 C CNN
 	1    5225 6625
